File: PCB + Schematic/plantMonitorAutoroute/plantMonitorAutoroute.kicad_sch (KiCad schematic)
At the start: 43 parts, among them J1 FTDI, J2 AT_ISP, SW1 AT_RESET, SW2 Power, SW3 BUTTON1, SW4 BUTTON2, U1 ATmega328P-A, U2 Ra-01, U3 BME280, U4 TLC555xPS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

Commit message: PCB!
Parts:
- added C17: 1 nF, symbol Device:C_Small
- added Q1: DMN1019USN-13, Package_TO_SOT_SMD:SC-59_Handsoldering, symbol Transistor_FET:DMN1019USN-13
- added R10: 10, Resistor_SMD:R_0402_1005Metric, symbol Device:R
- added R11, R12: 1 M, Resistor_SMD:R_0402_1005Metric, symbol Device:R_Small
- added R9: 10 K, Resistor_SMD:R_0402_1005Metric, symbol Device:R
Connections:
- net +3.3V: now also C17.1, R11.2
- net GND: now also C14.1, C15.1, R7.1, C17.2, Q1.1 (S), R12.1, R9.2; no longer U4.1 (GND)
- net VOLT: now reaches U1.24 (PC1)
- net VOLT: now also R11.1, R12.2
- net SOIL_FET: now reaches U1.9 (PD5)
- net SOIL_FET: now also R10.2
- new net: Q1.2 (G), R10.1, R9.1
- new net: Q1.3 (D), U4.1 (GND)
Other:
- moved on the sheet: AE1, BT1, C10, C11, C12, C13, C14, C15, C16, C8, C9, D2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
