File: PCB + Schematic/plantMonitorCopy/plantMonitorCopy.kicad_pcb (KiCad board)
At the start: 2 copper layers, 23.2 x 124.7 mm, 48 parts, among them J1 FTDI, J2 AT_ISP, J3 FTDI, Q1 DMN1019USN-13, SW1 AT_RESET, SW2 Power, SW3 BUTTON1, SW4 BUTTON2, U1 ATmega328P-A, U2 Ra-01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

Commit message: PCB
Parts:
- added H1: MountingHole, MountingHole:MountingHole_2.2mm_M2, F.Cu at (272.8, 141.5)
- added H4: MountingHole, MountingHole:MountingHole_2.2mm_M2, F.Cu at (272.8, 147.4)
- moved D1 101.0 mm to (355.1, 38.0)
- moved R2 101.0 mm to (355.3, 39.2)
- moved C12 90.0 mm to (173.2, 67.1)
- moved C13 90.0 mm to (164.7, 68.6)
- moved C16 90.0 mm to (173.3, 70.5)
- moved R5 90.0 mm to (173.9, 69.0)
- moved R6 90.0 mm to (172.8, 69.0)
- moved R7 90.0 mm to (165.7, 73.0)
- moved R8 90.0 mm to (166.2, 71.5)
- moved U4 90.0 mm to (168.8, 69.1)
- moved C15 90.0 mm to (166.8, 73.1)
- moved D2 90.0 mm to (168.2, 72.5)
- moved J2 68.6 mm to (322.2, 88.4)
- moved R1 44.2 mm to (214.5, 64.1)
- moved SW1 44.2 mm to (209.0, 63.0)
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Routing:
- net +3.3V: track 185.3 -> 17.7 mm, vias 6 -> 0
- net GND: track 172.8 -> 14.0 mm, vias 5 -> 0
- net MISO: track 53.9 -> 0.00 mm, vias 3 -> 0
- net SCL: track 52.1 -> 0.49 mm, vias 2 -> 0
- net CS: track 48.5 -> 0.00 mm, vias 2 -> 0
- net DIO0: track 44.8 -> 0.00 mm, vias 2 -> 0
- net SCK: track 44.8 -> 0.00 mm, vias 2 -> 0
- net LORA_RST: track 43.1 -> 0.00 mm, vias 2 -> 0
- net MOSI: track 42.7 -> 0.00 mm, vias 1 -> 0
- net SDA: track 42.2 -> 0.54 mm
- net RESET: track 34.1 -> 0.00 mm, vias 2 -> 0
- net RX: track 30.2 -> 0.00 mm, vias 3 -> 0
- net BUTTON2: track 27.1 -> 0.00 mm, vias 2 -> 0
- net BUTTON1: track 19.5 -> 0.00 mm, vias 2 -> 0
- net TX: track 12.1 -> 0.00 mm, vias 1 -> 0
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Other:
- board size 23.2 x 124.7 mm -> 25.7 x 126 mm

Commit message: PCB
Parts:
- J1: moved to B.Cu
- J3: value FTDI -> GPIO; footprint Connector_PinHeader_2.54mm:PinHeader_1x06_P2.54mm_Vertical -> Connector_PinHeader_2.54mm:PinHeader_1x05_P2.54mm_Vertical; moved to B.Cu
- moved D1 119.1 mm to (245.6, 85.0), turned to 180 degrees
- moved R2 118.7 mm to (245.3, 83.7), turned to 0 degrees
- moved C13 87.3 mm to (241.5, 109.9), turned to -90 degrees
- moved C12 86.6 mm to (250.2, 106.8)
- moved C15 86.4 mm to (243.7, 112.4)
- moved C16 86.4 mm to (250.2, 109.8)
- moved D2 86.4 mm to (245.1, 111.8)
- moved R5 86.4 mm to (250.8, 108.3)
- moved R6 86.4 mm to (249.7, 108.3)
- moved R7 86.4 mm to (242.6, 112.4)
- moved R8 86.4 mm to (243.1, 110.8)
- moved U4 86.4 mm to (245.7, 108.4)
- moved J2 64.7 mm to (257.9, 80.7), turned to 90 degrees
- moved SW3 60.9 mm to (261.1, 90.3)
- moved SW1 60.9 mm to (261.1, 94.7)
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Connections:
- C14 pad 1: GND -> Net-(D2-A)
- J3 pad 1: unconnected-(J3-Pin_1-Pad1) -> SDA
- J3 pad 2: unconnected-(J3-Pin_2-Pad2) -> SCL
- J3 pad 3: unconnected-(J3-Pin_3-Pad3) -> A3
- J3 pad 4: unconnected-(J3-Pin_4-Pad4) -> A2
- J3 pad 5: unconnected-(J3-Pin_5-Pad5) -> D2
- U1 pad 25: unconnected-(U1-PC2-Pad25) -> A2
- U1 pad 26: unconnected-(U1-PC3-Pad26) -> A3
- U1 pad 32: unconnected-(U1-PD2-Pad32) -> D2
Routing:
- net XTAL2: track 0.00 -> 29.9 mm
- net XTAL1: track 0.00 -> 20.4 mm
- net +3.3V: track 17.7 -> 35.8 mm
- net TRIG: track 0.00 -> 14.4 mm, vias 0 -> 2
- net OUT: track 0.00 -> 10.5 mm, vias 0 -> 2
- net GND: track 14.0 -> 24.2 mm, vias 0 -> 4
- net Net-(Q1-D): track 0.00 -> 6.09 mm
- net Net-(U4-DIS): track 0.00 -> 3.06 mm
- net Net-(D2-A): track 0.00 -> 2.94 mm
- net Net-(Q1-G): track 0.00 -> 2.85 mm
- net SOIL: track 0.00 -> 2.65 mm
- net VOLT: track 0.00 -> 2.58 mm
- net COUT: track 0.00 -> 2.07 mm
- net SCL: track 0.49 -> 2.07 mm
- net SDA: track 0.54 -> 2.09 mm
Other:
- outline, holes or cut-outs redrawn
