File: PCB + Schematic/plantMonitorCopy/plantMonitorCopy.kicad_sch (KiCad schematic)
At the start: 50 parts, among them J1 FTDI, J2 AT_ISP, J3 FTDI, Q1 DMN1019USN-13, SW1 AT_RESET, SW2 Power, SW3 BUTTON1, SW4 BUTTON2, U1 ATmega328P-A, U2 Ra-01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

Commit message: PCB
Parts:
- removed J3: FTDI, Connector_PinHeader_2.54mm:PinHeader_1x06_P2.54mm_Vertical, symbol Connector_Generic:Conn_01x06
- added J3: GPIO, Connector_PinHeader_2.54mm:PinHeader_1x05_P2.54mm_Vertical, symbol Connector_Generic:Conn_01x05
Connections:
- net GND: now also C14.2; no longer C14.1
- net SCL: now also J3.2 (Pin_2)
- net SDA: now also J3.1 (Pin_1)
- net at D2.2 (A), R8.1: now also C14.1; no longer C14.2
- net A2: now reaches U1.25 (PC2)
- net A2: now also J3.4 (Pin_4)
- net A3: now reaches U1.26 (PC3)
- net A3: now also J3.3 (Pin_3)
- net D2: now reaches U1.32 (PD2)
- net D2: now also J3.5 (Pin_5)
Other:
- moved on the sheet: C14
