File: PCB + Schematic/plantMonitor/plantMonitorCopy.kicad_sch (KiCad schematic)
At the start: 50 parts, among them J1 FTDI, J2 AT_ISP, J3 GPIO, Q1 DMN1019USN-13, SW1 AT_RESET, SW2 Power, SW3 BUTTON1, SW4 BUTTON2, U1 ATmega328P-A, U2 Ra-01, U3 BME280, U4 TLC555xPS, Y1 8MHz

Commit message: Part finding
Parts:
- removed C13: 100 nF, Capacitor_SMD:C_0402_1005Metric, symbol Device:C_Small
- removed C15: 1 nF, Capacitor_SMD:C_0402_1005Metric, symbol Device:C_Small
- removed R10: 10, Resistor_SMD:R_0402_1005Metric, symbol Device:R
- removed R11: 1 M, Resistor_SMD:R_0402_1005Metric, symbol Device:R_Small
- removed R9: 10 K, Resistor_SMD:R_0402_1005Metric, symbol Device:R
- removed SW4: BUTTON2, Button_Switch_SMD:SW_SPST_CK_RS282G05A3, symbol Switch:SW_Push
- removed U4: TLC555xPS, Package_SO:VSSOP-8_3.0x3.0mm_P0.65mm, symbol Timer:TLC555xPS
- added C14: 100 nF, Capacitor_SMD:C_0402_1005Metric, symbol symbols:C_Small
- added C16: 1 nF, Capacitor_SMD:C_0402_1005Metric, symbol Device:C_Small
- added R4: 1 M, Resistor_SMD:R_0402_1005Metric, symbol Device:R_Small
- added R7, R8: 10 K, Resistor_SMD:R_0402_1005Metric, symbol Device:R_Small
- added SW2: BUTTON1, Button_Switch_SMD:SW_SPST_CK_RS282G05A3, symbol Switch:SW_Push
- added U5: TLC555CDR, Package_SO:SOIC-8_3.9x4.9mm_P1.27mm, symbol Timer:TLC555xD
- C13: renamed from C12; footprint Capacitor_SMD:C_0402_1005Metric -> Capacitor_SMD:C_0603_1608Metric; LCSC (none) -> C1620
- C15: renamed from C16; LCSC (none) -> C15195
- C6: renamed from C7; LCSC (none) -> C1555
- C7: renamed from C6; LCSC (none) -> C1555
- C8: renamed from C17; LCSC (none) -> C1523
- D2: value SM4007 -> MCL103A; LCSC (none) -> C142609
- R10: renamed from R5; LCSC (none) -> C25104
- R11: renamed from R8; LCSC (none) -> C25744
- R5: renamed from R12; LCSC (none) -> C26083
- R9: renamed from R6; LCSC (none) -> C25867
- SW1: value AT_RESET -> BUTTON2; LCSC (none) -> C2888954
- SW3: value BUTTON1 -> RESET; LCSC (none) -> C2888954
- U3: renamed from U1; LCSC (none) -> C14877
- renumbered C11 to C1, C4 to C10, C1 to C11, C2 to C12, C14 to C17, C10 to C2, C8 to C3, C9 to C4, C3 to C9, H4 to H1, H1 to H2, H2 to H4, J2 to J1, J1 to J2, R4 to R1, R7 to R12, R1 to R6, SW2 to SW4, U3 to U1
Connections:
- net +3.3V: now also SW1.2, C14.1, R4.2, SW2.2, U5.4 (R), U5.8 (VCC); no longer SW3.2
- net BUTTON1: now also SW2.1; no longer SW3.1
- net BUTTON2: now also SW1.1
- net COUT: now also U5.5 (CV)
- net GND: now also SW3.2, C14.2, C16.2, R7.2; no longer SW1.2
- net OUT: now also U5.3 (Q)
- net RESET: now also SW3.1; no longer SW1.1
- net SOIL: now also C16.1
- net SOIL_FET: now also R8.2
- net TRIG: now also U5.2 (TR), U5.6 (THR)
- net VOLT: now also R4.1
- net at R10.1, R9.1: now also U5.7 (DIS)
- net at Q1.2 (G): now also R7.1, R8.1
- net at Q1.3 (D): now also U5.1 (GND)
