File: PCB + Schematic/groundMonitor/groundMonitor.kicad_pcb (KiCad board)
At the start: 2 copper layers, 22 parts, among them J1 FTDI, J2 Header, J3 5-12 V, J4 USB-C, J5 Power, SW1 EN, SW2 Boot, U1 ESP32-C3-MINI-1-N4, U2 AMS1117-3.3, U3 Ra-01

Commit message: More PCB
Parts:
- removed AE1: Antenna, Connector_PinHeader_2.54mm:PinHeader_1x01_P2.54mm_Vertical
- added AE2: Antenna, Connector_Coaxial:SMA_Amphenol_132289_EdgeMount, F.Cu at (219.8, 118.5)
- added H1: Hole, MountingHole:MountingHole_3.2mm_M3, F.Cu at (216.9, 108.5)
- added H2: Hole, MountingHole:MountingHole_3.2mm_M3, F.Cu at (194.4, 90.0)
- added H3: Hole, MountingHole:MountingHole_3.2mm_M3, F.Cu at (220.9, 90.0)
- added H4: Hole, MountingHole:MountingHole_3.2mm_M3, F.Cu at (200.7, 126.6)
- moved R4 80.8 mm to (214.6, 103.8), turned to 90 degrees
- moved C2 79.3 mm to (208.9, 126.8)
- moved C4 79.1 mm to (215.4, 115.2), turned to 90 degrees
- moved J2 78.9 mm to (193.9, 121.0), turned to 180 degrees
- moved J1 78.3 mm to (221.4, 95.4)
- moved C7 78.1 mm to (215.4, 118.4), turned to -90 degrees
- moved C1 77.6 mm to (205.6, 126.8), turned to 180 degrees
- moved C3 72.8 mm to (200.5, 130.9)
- moved R1 72.6 mm to (198.5, 130.6), turned to 90 degrees
- moved U3 69.7 mm to (205.1, 114.3), turned to 180 degrees
- moved R3 69.3 mm to (195.6, 131.1), turned to 180 degrees
- moved J3 66.3 mm to (216.3, 126.5), turned to 90 degrees
- moved SW2 65.8 mm to (216.3, 96.8), turned to -90 degrees
- moved C6 60.5 mm to (199.3, 93.7), turned to 90 degrees
- moved C5 58.7 mm to (197.6, 93.7), turned to 90 degrees
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Connections:
- J2 pad 2: SCL -> SS
- J2 pad 3: SDA -> MOSI
- J2 pad 4: SS -> MISO
- J2 pad 5: MISO -> SCK
- J2 pad 6: SCK -> SCL
- J2 pad 7: MOSI -> SDA
- U3 pad 15: CS -> SS
Routing:
- net GND: track 0.00 -> 87.5 mm
- net VCC: track 0.00 -> 39.3 mm
- net +3.3V: track 0.00 -> 36.9 mm, vias 0 -> 2
- net SCK: track 0.00 -> 25.1 mm, vias 0 -> 2
- net SS: track 0.00 -> 24.0 mm
- net MISO: track 0.00 -> 23.6 mm, vias 0 -> 2
- net MOSI: track 0.00 -> 22.3 mm
- net SDA: track 0.00 -> 19.3 mm, vias 0 -> 2
- net SCL: track 0.00 -> 17.4 mm
- net unconnected-(J4-SHIELD-PadS1): track 0.00 -> 17.0 mm
- net A0: track 0.00 -> 10.6 mm, vias 0 -> 1
- net BOOT: track 0.00 -> 9.02 mm, vias 0 -> 2
- net Net-(AE2-A): track 0.00 -> 7.90 mm
- net D7: track 0.00 -> 6.95 mm, vias 0 -> 2
- net EN: track 0.00 -> 6.26 mm
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- added copper zone on B.Cu, net GND
- added copper zone on F.Cu, net GND
Other:
- board outline added: 31.2 x 52.3 mm

Commit message: More PCB
Parts:
- moved H3 0.92 mm to (217.2, 109.3)
- renumbered AE2 to AE1, C5 to C1, C6 to C2, C4 to C3, C7 to C4, C1 to C5, C2 to C6, C3 to C7, D2 to D1, H2 to H1, H3 to H2, H1 to H3, R4 to R1, R3 to R2, R1 to R3, SW2 to SW1, SW1 to SW2, U3 to U2, U2 to U3
Routing:
- net D+: track 2.56 -> 49.3 mm
- net +3.3V: track 36.9 -> 78.8 mm, vias 2 -> 3
- net EN: track 6.26 -> 44.3 mm, vias 0 -> 1
- net D-: track 2.56 -> 40.6 mm
- net GND: track 87.5 -> 123.3 mm, vias 0 -> 36
- net BOOT: track 9.02 -> 30.8 mm
- net A1: track 0.00 -> 10.9 mm, vias 0 -> 1
- net RX: track 0.00 -> 8.95 mm
- net TX: track 0.00 -> 8.58 mm
- net MISO: track 23.6 -> 26.0 mm
- net SS: track 24.0 -> 26.1 mm
- net SCL: track 17.4 -> 15.3 mm
- net MOSI: track 22.3 -> 24.0 mm
- net SDA: track 19.3 -> 18.2 mm
- net SCK: track 25.1 -> 26.1 mm
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Other:
- board text added: "3V3"
- board text added: "A0"
- board text added: "A1"
- board text added: "BOOT"
- board text added: "EN"
- board text added: "GND"
- board text added: "MISO"
- board text added: "MOSI"
- board text added: "NC"
- board text added: "Plant Monitor v1"
- board text added: "Plant Monitor v1.0 Designed by Charles Nicholson, July 2024 https://github.com/crnicholson/Plant-Monitor Licensed under CERN-OHL-S-2.0"
- board text added: "RX"
- board text added: "SCK"
- board text added: "SCL"
- board text added: "SDA"
- board text added: "SS"
- board text added: "TX"
- board text added: "VIN"
- board text added: "VIN: 5-12 V"

Commit message: PCB!
Connections:
- J2 pad 8: A0 -> LORA_RST
- J2 pad 9: A1 -> DIO0
- U1 pad 12: A0 -> LORA_RST
- U1 pad 13: A1 -> DIO0
Routing:
- net DIO0: track 0.00 -> 60.6 mm, vias 0 -> 2
- net LORA_RST: track 0.00 -> 54.4 mm, vias 0 -> 3
- net A1: track 10.9 -> 0.00 mm, vias 1 -> 0
- net A0: track 9.68 -> 0.00 mm, vias 1 -> 0
- net +3.3V: track 78.8 -> 79.7 mm

Commit message: PCB stuff, file org
Other:
- board text added: "JLCJLCJLCJLC"
Changed lines of the file:
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@@
+		)
+	)
+	(gr_text "JLCJLCJLCJLC"
+		(at 213.0044 89.408 0)
+		(layer "B.SilkS")
+		(effects
+			(font
+				(size 1 1)
+				(thickness 0.15)
+			)
+			(justify left bottom mirror)
 		)
 	)
@@
 	)
 	(gr_text "3V3"
-		(at 219.964 106.68 90)
+		(at 220.1672 106.7308 90)
 		(layer "B.SilkS")
 		(effects
@@
 		(layers "F&B.Cu")
 		(hatch edge 0.5)
-		(connect_pads
+		(connect_pads yes
 			(clearance 0.5)
 		)

Commit message: Edit README
Parts:
- U1: value ESP32-C3-MINI-1-N4 -> ESP32-C3-MINI-1-H4
Changed lines of the file:
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@@
 			)
 		)
-		(property "Value" "ESP32-C3-MINI-1-N4"
+		(property "Value" "ESP32-C3-MINI-1-H4"
 			(at 0 0 0)
 			(unlocked yes)
@@
 				)
 			)
+		)
+		(property "LCSC" "C2934569 "
+			(at 0 0 0)
+			(unlocked yes)
+			(layer "F.Fab")
+			(hide yes)
+			(effects
+				(font
+					(size 1 1)
+					(thickness 0.15)
+				)
+			)
