File: PCB + Schematic/groundMonitor/groundMonitor.kicad_sch (KiCad schematic)
At the start: 16 parts, among them J1 FTDI, J2 FTDI, SW1 Boot, SW2 Boot, SW3 Reset, SW4 Reset, U1 ESP32-MINI-1-N4, U2 ESP32-C3-WROOM-02-N4, U3 ESP32-C3-MINI-1-N4

Commit message: PCB
Parts:
- removed J2: FTDI, symbol Connector_Generic:Conn_01x06
- removed SW3, SW4: Reset, symbol Switch:SW_Push
- removed U1: ESP32-MINI-1-N4, ESP32-MINI-1-N4:XCVR_ESP32-MINI-1-N4, symbol ESP32-MINI-1-N4:ESP32-MINI-1-N4
- removed U2: ESP32-C3-WROOM-02-N4, ESP32-C3-WROOM-02-N4:MODULE_ESP32-C3-WROOM-02-H4, symbol ESP32-C3-WROOM-02-N4:ESP32-C3-WROOM-02-N4
- removed U3: ESP32-C3-MINI-1-N4, ESP32-C3-MINI-1_EXP, symbol ESP32-MINI-1-N4-New:ESP32-C3-MINI-1-N4
- added AE1: Antenna, Connector_PinHeader_2.54mm:PinHeader_1x01_P2.54mm_Vertical, symbol Connector_Generic:Conn_01x01
- added C7: 100 nF, Capacitor_SMD:C_0603_1608Metric, symbol Device:C_Small
- added D2: RED, LED_SMD:LED_0603_1608Metric, symbol Device:LED_Small
- added J2: Header, Connector_PinHeader_2.54mm:PinHeader_1x11_P2.54mm_Vertical, symbol Connector_Generic:Conn_01x11
- added J3: 5-12 V, Connector_BarrelJack:BarrelJack_Horizontal, symbol Connector:Barrel_Jack_Switch
- added J4: USB-C, Connector_USB:USB_C_Receptacle_GCT_USB4105-xx-A_16P_TopMnt_Horizontal, symbol Connector:USB_C_Receptacle_USB2.0
- added J5: Power, Connector_PinHeader_2.54mm:PinHeader_1x03_P2.54mm_Vertical, symbol Connector_Generic:Conn_01x03
- added R3: 5.1 K, Resistor_SMD:R_0402_1005Metric, symbol Device:R_Small
- added R4: 1 K, Resistor_SMD:R_0402_1005Metric, symbol Device:R_Small
- added U1: ESP32-C3-MINI-1-N4, ESP32-C3-MINI-1-N4:ESP32-C3-MINI-1_EXP, symbol ESP32-MINI-1-N4-New:ESP32-C3-MINI-1-N4
- added U2: AMS1117-3.3, Package_TO_SOT_SMD:SOT-223-3_TabPin2, symbol Regulator_Linear:AMS1117-3.3
- added U3: Ra-01, RF_Module:Ai-Thinker-Ra-01-LoRa, symbol RF_Module:Ai-Thinker-Ra-01
- C1, C5: value 100 nF -> 10 uF; footprint (none) -> Capacitor_SMD:C_0603_1608Metric; LCSC (none) -> C19702
- C2, C6: value 10 uF -> 100 nF; footprint (none) -> Capacitor_SMD:C_0603_1608Metric; LCSC (none) -> C14663
- C3: footprint (none) -> Capacitor_SMD:C_0603_1608Metric; LCSC (none) -> C14663
- C4: footprint (none) -> Capacitor_SMD:C_0603_1608Metric; LCSC (none) -> C19702
- J1: footprint (none) -> Connector_PinHeader_2.54mm:PinHeader_1x06_P2.54mm_Vertical
- R1: value 10 K -> 5.1 K; footprint (none) -> Resistor_SMD:R_0402_1005Metric; LCSC (none) -> C25905
- SW1: value Boot -> EN; footprint (none) -> Button_Switch_SMD:SW_SPST_CK_RS282G05A3; LCSC (none) -> C2888954
- SW2: footprint (none) -> Button_Switch_SMD:SW_SPST_CK_RS282G05A3; LCSC (none) -> C2888954
Connections:
- net +3.3V: now also C2.1, C4.1, J1.6 (Pin_6), C7.1, J5.2 (Pin_2), U1.3 (3V3), U2.2 (VO), U3.3 (VDD); no longer R1.1
- net BOOT: now also J2.11 (Pin_11), U1.23 (IO9); no longer SW1.2
- net EN: now also SW1.2, J2.10 (Pin_10), U1.8 (EN)
- net GND: now also C1.1, R1.2, C7.2, D2.1 (K), J2.1 (Pin_1), J3.2, J3.3, J4.A1 (GND), J4.A12 (GND), J4.B1 (GND), J4.B12 (GND), J5.1 (Pin_1), R3.2, U1.1 (GND), U1.11 (GND), U1.14 (GND), U1.36 (GND), U1.37 (GND), U1.38 (GND), U1.39 (GND), U1.40 (GND), U1.41 (GND), U1.42 (GND), U1.43 (GND), U1.44 (GND), U1.45 (GND), U1.46 (GND), U1.47 (GND), U1.48 (GND), U1.49 (GND), U1.50 (GND), U1.51 (GND), U1.52 (GND), U1.53 (GND), U1.54 (GND), U1.55 (GND), U1.56 (GND), U1.57 (GND), U1.58 (GND), U1.59 (GND), U1.60 (GND), U1.61 (GND), U2.1 (GND), U3.16 (GND), U3.2 (GND), U3.9 (GND); no longer C1.2
- net RX: now also U1.30 (RXD0)
- net TX: now also U1.31 (TXD0)
- net VCC: now also C1.2, C3.1, J3.1, J4.A4 (VBUS), J4.A9 (VBUS), J4.B4 (VBUS), J4.B9 (VBUS), J5.3 (Pin_3), U2.3 (VI); no longer J1.6 (Pin_6)
- new net: D2.2 (A), R4.1
- new net: J4.B5 (CC2), R1.1
- new net: J4.A5 (CC1), R3.1
- new net: AE1.1 (Pin_1), U3.1 (ANT)
- new net A0: J2.8 (Pin_8), U1.12 (IO0)
- new net A1: J2.9 (Pin_9), U1.13 (IO1)
- new net CS: U3.15 (~{NSS})
- new net D+: J4.A6 (D+), J4.B6 (D+), U1.27 (IO19)
- new net D-: J4.A7 (D-), J4.B7 (D-), U1.26 (IO18)
- new net D7: R4.2, U1.21 (IO7)
- new net DIO0: U3.5 (DIO0)
- new net LORA_RST: U3.4 (~{RESET})
- new net MISO: J2.5 (Pin_5), U1.6 (IO3), U3.13 (MISO)
- new net MOSI: J2.7 (Pin_7), U1.18 (IO4), U3.14 (MOSI)
- new net SCK: J2.6 (Pin_6), U1.5 (IO2), U3.12 (SCK)
- new net SCL: J2.2 (Pin_2), U1.16 (IO10)
- new net SDA: J2.3 (Pin_3), U1.22 (IO8)
- new net SS: J2.4 (Pin_4), U1.19 (IO5)
Other:
- note added: "ESP32 module"
- note added: "Headers"
- note added: "LoRa module"
- note added: "Power"
- moved on the sheet: J1

Commit message: More PCB
Parts:
- removed AE1: Antenna, Connector_PinHeader_2.54mm:PinHeader_1x01_P2.54mm_Vertical, symbol Connector_Generic:Conn_01x01
- added AE2: Antenna, Connector_Coaxial:SMA_Amphenol_132289_EdgeMount, symbol Device:Antenna_Shield
- added H1, H2, H3, H4: Hole, MountingHole:MountingHole_3.2mm_M3, symbol Mechanical:MountingHole
Connections:
- net CS is gone; now on net SS: U3.15 (~{NSS})
- net GND: now also AE2.2 (Shield)
- net MISO: now also J2.4 (Pin_4); no longer J2.5 (Pin_5)
- net MOSI: now also J2.3 (Pin_3); no longer J2.7 (Pin_7)
- net SCK: now also J2.5 (Pin_5); no longer J2.6 (Pin_6)
- net SCL: now also J2.6 (Pin_6); no longer J2.2 (Pin_2)
- net SDA: now also J2.7 (Pin_7); no longer J2.3 (Pin_3)
- net SS: now also J2.2 (Pin_2); no longer J2.4 (Pin_4)
- net at U3.1 (ANT): now also AE2.1 (A)
Other:
- moved on the sheet: C4, C7, U3

Commit message: More PCB
Parts:
- renumbered AE2 to AE1, C5 to C1, C6 to C2, C4 to C3, C7 to C4, C1 to C5, C2 to C6, C3 to C7, D2 to D1, H2 to H1, H3 to H2, H1 to H3, R4 to R1, R3 to R2, R1 to R3, SW2 to SW1, SW1 to SW2, U3 to U2, U2 to U3
Other:
- note added: "Mounting holes"
- moved on the sheet: H1, H2, H3, H4
Changed lines of the file:
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@@
 	)
 	(rectangle
+		(start 247.65 129.54)
+		(end 266.7 162.56)
+		(stroke
+			(width 0)
+			(type default)
+		)
+		(fill
+			(type none)
+		)
+	)
+	(rectangle
 		(start 15.24 100.33)
 		(end 101.6 195.58)
@@
 		)
 	)
+	(text "Mounting holes"
+		(exclude_from_sim no)
+		(at 257.175 159.385 0)
+		(effects
+			(font
+				(size 1.27 1.27)
+			)
+		)
+	)
 	(text "LoRa module"
 		(exclude_from_sim no)
@@
 	(symbol
 		(lib_id "Mechanical:MountingHole")
-		(at 190.5 96.52 0)
+		(at 252.73 147.32 0)
 		(unit 1)
 		(exclude_from_sim yes)
@@
 		(dnp no)
 		(fields_autoplaced yes)
-		(property "Reference" "H3"
-			(at 193.04 95.2499 0)
+		(property "Reference" "H2"
+			(at 255.27 146.0499 0)
 			(effects
 				(font
@@
 		)
 		(property "Value" "Hole"
-			(at 193.04 97.7899 0)
+			(at 255.27 148.5899 0)
 			(effects
 				(font
@@
 		)
 		(property "Footprint" "MountingHole:MountingHole_3.2mm_M3"
-			(at 190.5 96.52 0)
+			(at 252.73 147.32 0)
 			(effects
 				(font
@@
 		)
 		(property "Datasheet" "~"
-			(at 190.5 96.52 0)
+			(at 252.73 147.32 0)
 			(effects
 				(font
@@
 		)
 		(property "Description" "Mounting Hole without connection"
-			(at 190.5 96.52 0)
+			(at 252.73 147.32 0)
 			(effects
 				(font
@@
 			(project "groundMonitor"
 				(path "/c28ff6ee-0862-40d7-9eed-e06e2f3ba893"
-					(reference "H3")
+					(reference "H2")
 					(unit 1)
 				)
@@
 		(dnp no)
 		(fields_autoplaced yes)
-		(property "Reference" "D2"
+		(property "Reference" "D1"
 			(at 24.13 148.5264 90)
 			(effects
@@
 			(project "groundMonitor"
 				(path "/c28ff6ee-0862-40d7-9eed-e06e2f3ba893"
-					(reference "D2")
+					(reference "D1")
 					(unit 1)
 				)
@@
 		(dnp no)
 		(fields_autoplaced yes)
-		(property "Reference" "R1"
+		(property "Reference" "R3"
 			(at 142.24 162.5599 0)
 			(effects
@@
 			(project "groundMonitor"
 				(path "/c28ff6ee-0862-40d7-9eed-e06e2f3ba893"
-					(reference "R1")
+					(reference "R3")
 					(unit 1)
 				)
@@
 		(dnp no)
 		(fields_autoplaced yes)
-		(property "Reference" "SW1"
+		(property "Reference" "SW2"
 			(at 35.56 176.5299 90)
 			(effects
@@
 			(project "groundMonitor"
 				(path "/c28ff6ee-0862-40d7-9eed-e06e2f3ba893"
-					(reference "SW1")
+					(reference "SW2")
 					(unit 1)
 				)
@@
 	(symbol
 		(lib_id "Mechanical:MountingHole")
-		(at 190.5 90.17 0)
+		(at 252.73 140.97 0)
 		(unit 1)
 		(exclude_from_sim yes)
@@
 		(dnp no)
 		(fields_autoplaced yes)
-		(property "Reference" "H2"
-			(at 193.04 88.8999 0)
+		(property "Reference" "H1"
+			(at 255.27 139.6999 0)
 			(effects
 				(font
@@
 		)
 		(property "Value" "Hole"
-			(at 193.04 91.4399 0)
+			(at 255.27 142.2399 0)
 			(effects
 				(font
@@
 		)
 		(property "Footprint" "MountingHole:MountingHole_3.2mm_M3"
-			(at 190.5 90.17 0)
+			(at 252.73 140.97 0)
 			(effects
 				(font
@@
 		)
 		(property "Datasheet" "~"
-			(at 190.5 90.17 0)
+			(at 252.73 140.97 0)
 			(effects
 				(font
@@
 		)
 		(property "Description" "Mounting Hole without connection"
-			(at 190.5 90.17 0)
+			(at 252.73 140.97 0)
 			(effects
 				(font
@@
 			(project "groundMonitor"
 				(path "/c28ff6ee-0862-40d7-9eed-e06e2f3ba893"
-					(reference "H2")
+					(reference "H1")
 					(unit 1)
 				)
@@
 	(symbol
 		(lib_id "Mechanical:MountingHole")
-		(at 190.5 102.87 0)
+		(at 252.73 153.67 0)
 		(unit 1)
 		(exclude_from_sim yes)
@@
 		(fields_autoplaced yes)
 		(property "Reference" "H4"
-			(at 193.04 101.5999 0)
+			(at 255.27 152.3999 0)
 			(effects
 				(font
@@
 		)
 		(property "Value" "Hole"
-			(at 193.04 104.1399 0)
+			(at 255.27 154.9399 0)
 			(effects
 				(font
@@
 		)
 		(property "Footprint" "MountingHole:MountingHole_3.2mm_M3"
-			(at 190.5 102.87 0)
+			(at 252.73 153.67 0)
 			(effects
 				(font
@@
 		)
 		(property "Datasheet" "~"
-			(at 190.5 102.87 0)
+			(at 252.73 153.67 0)
 			(effects
 				(font
@@
 		)
 		(property "Description" "Mounting Hole without connection"
-			(at 190.5 102.87 0)
+			(at 252.73 153.67 0)
 			(effects
 				(font
@@
 		(dnp no)
 		(fields_autoplaced yes)
-		(property "Reference" "C5"
+		(property "Reference" "C1"
 			(at 36.83 119.3862 0)
 			(effects
@@
 			(project "groundMonitor"
 				(path "/c28ff6ee-0862-40d7-9eed-e06e2f3ba893"
-					(reference "C5")
+					(reference "C1")
 					(unit 1)
 				)
@@
 		(dnp no)
 		(fields_autoplaced yes)
-		(property "Reference" "C6"
+		(property "Reference" "C2"
 			(at 24.13 119.3862 0)
 			(effects
@@
 			(project "groundMonitor"
 				(path "/c28ff6ee-0862-40d7-9eed-e06e2f3ba893"
-					(reference "C6")
+					(reference "C2")
 					(unit 1)
 				)
@@
 		(dnp no)
 		(fields_autoplaced yes)
-		(property "Reference" "U2"
+		(property "Reference" "U3"
 			(at 124.46 116.84 0)
 			(effects
@@
 			(project "groundMonitor"
 				(path "/c28ff6ee-0862-40d7-9eed-e06e2f3ba893"
-					(reference "U2")
+					(reference "U3")
 					(unit 1)
 				)
@@
 		(dnp no)
 		(fields_autoplaced yes)
-		(property "Reference" "C3"
+		(property "Reference" "C7"
 			(at 156.21 149.8662 0)
 			(effects
@@
 			(project "groundMonitor"
 				(path "/c28ff6ee-0862-40d7-9eed-e06e2f3ba893"
-					(reference "C3")
+					(reference "C7")
 					(unit 1)
 				)
@@
 		(dnp no)
 		(fields_autoplaced yes)
-		(property "Reference" "C1"
+		(property "Reference" "C5"
 			(at 111.76 128.2638 0)
 			(effects
@@
 			(project "groundMonitor"
 				(path "/c28ff6ee-0862-40d7-9eed-e06e2f3ba893"
-					(reference "C1")
+					(reference "C5")
 					(unit 1)
 				)
@@
 		(dnp no)
 		(fields_autoplaced yes)
-		(property "Reference" "AE2"
+		(property "Reference" "AE1"
 			(at 234.95 121.2849 0)
 			(effects
@@
 			(project "groundMonitor"
 				(path "/c28ff6ee-0862-40d7-9eed-e06e2f3ba893"
-					(reference "AE2")
+					(reference "AE1")
 					(unit 1)
 				)
@@
 		(dnp no)
 		(fields_autoplaced yes)
-		(property "Reference" "C7"
+		(property "Reference" "C4"
 			(at 193.04 137.1662 0)
 			(effects
@@
 			(project "groundMonitor"
 				(path "/c28ff6ee-0862-40d7-9eed-e06e2f3ba893"
-					(reference "C7")
+					(reference "C4")
 					(unit 1)
 				)
@@
 		(dnp no)
 		(fields_autoplaced yes)
-		(property "Reference" "R4"
+		(property "Reference" "R1"
 			(at 24.13 143.5099 0)
 			(effects
@@
 			(project "groundMonitor"
 				(path "/c28ff6ee-0862-40d7-9eed-e06e2f3ba893"
-					(reference "R4")
+					(reference "R1")
 					(unit 1)
 				)
@@
 	(symbol
 		(lib_id "Mechanical:MountingHole")
-		(at 190.5 83.82 0)
+		(at 252.73 134.62 0)
 		(unit 1)
 		(exclude_from_sim yes)
@@
 		(dnp no)
 		(fields_autoplaced yes)
-		(property "Reference" "H1"
-			(at 193.04 82.5499 0)
+		(property "Reference" "H3"
+			(at 255.27 133.3499 0)
 			(effects
 				(font
@@
 		)
 		(property "Value" "Hole"
-			(at 193.04 85.0899 0)
+			(at 255.27 135.8899 0)
 			(effects
 				(font
@@
 		)
 		(property "Footprint" "MountingHole:MountingHole_3.2mm_M3"
-			(at 190.5 83.82 0)
+			(at 252.73 134.62 0)
 			(effects
 				(font
@@
 		)
 		(property "Datasheet" "~"
-			(at 190.5 83.82 0)
+			(at 252.73 134.62 0)
 			(effects
 				(font
@@
 		)
 		(property "Description" "Mounting Hole without connection"
-			(at 190.5 83.82 0)
+			(at 252.73 134.62 0)
 			(effects
 				(font
@@
 			(project "groundMonitor"
 				(path "/c28ff6ee-0862-40d7-9eed-e06e2f3ba893"
-					(reference "H1")
+					(reference "H3")
 					(unit 1)
 				)
@@
 		(dnp no)
 		(fields_autoplaced yes)
-		(property "Reference" "R3"
+		(property "Reference" "R2"
 			(at 152.4 162.5599 0)
 			(effects
@@
 			(project "groundMonitor"
 				(path "/c28ff6ee-0862-40d7-9eed-e06e2f3ba893"
-					(reference "R3")
+					(reference "R2")
 					(unit 1)
 				)
@@
 		(dnp no)
 		(fields_autoplaced yes)
-		(property "Reference" "C4"
+		(property "Reference" "C3"
 			(at 181.61 137.1662 0)
 			(effects
@@
 			(project "groundMonitor"
 				(path "/c28ff6ee-0862-40d7-9eed-e06e2f3ba893"
-					(reference "C4")
+					(reference "C3")
 					(unit 1)
 				)
@@
 		(dnp no)
 		(fields_autoplaced yes)
-		(property "Reference" "U3"
+		(property "Reference" "U2"
 			(at 219.3641 153.67 0)
 			(effects
@@
 			(project "groundMonitor"
 				(path "/c28ff6ee-0862-40d7-9eed-e06e2f3ba893"
-					(reference "U3")
+					(reference "U2")
 					(unit 1)
 				)
@@
 		(dnp no)
 		(fields_autoplaced yes)
-		(property "Reference" "C2"
+		(property "Reference" "C6"
 			(at 137.16 125.7362 0)
 			(effects
@@
 			(project "groundMonitor"
 				(path "/c28ff6ee-0862-40d7-9eed-e06e2f3ba893"
-					(reference "C2")
+					(reference "C6")
 					(unit 1)
 				)
@@
 		(dnp no)
 		(fields_autoplaced yes)
-		(property "Reference" "SW2"
+		(property "Reference" "SW1"
 			(at 24.13 176.5299 90)
 			(effects
@@
 			(project "groundMonitor"
 				(path "/c28ff6ee-0862-40d7-9eed-e06e2f3ba893"
-					(reference "SW2")
+					(reference "SW1")
 					(unit 1)
 				)

Commit message: PCB!
Connections:
- net A0 is gone; now on net LORA_RST: J2.8 (Pin_8), U1.12 (IO0)
- net A1 is gone; now on net DIO0: J2.9 (Pin_9), U1.13 (IO1)
Changed lines of the file:
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@@
 	(wire
 		(pts
-			(xy 41.91 138.43) (xy 50.8 138.43)
+			(xy 35.56 138.43) (xy 50.8 138.43)
 		)
 		(stroke
@@
 		)
 	)
+	(global_label "LORA_RST"
+		(shape input)
+		(at 26.67 67.31 0)
+		(fields_autoplaced yes)
+		(effects
+			(font
+				(size 1.27 1.27)
+			)
+			(justify left)
+		)
+		(property "Intersheetrefs" "${INTERSHEET_REFS}"
+			(at 38.7871 67.31 0)
+			(effects
+				(font
+					(size 1.27 1.27)
+				)
+				(justify left)
+				(hide yes)
+			)
+		)
+	)
 	(global_label "BOOT"
 		(shape input)
@@
 		)
 	)
+	(global_label "DIO0"
+		(shape input)
+		(at 26.67 64.77 0)
+		(fields_autoplaced yes)
+		(effects
+			(font
+				(size 1.27 1.27)
+			)
+			(justify left)
+		)
+		(property "Intersheetrefs" "${INTERSHEET_REFS}"
+			(at 34.07 64.77 0)
+			(effects
+				(font
+					(size 1.27 1.27)
+				)
+				(justify left)
+				(hide yes)
+			)
+		)
+	)
 	(global_label "D7"
 		(shape input)
@@
 		)
 	)
+	(global_label "LORA_RST"
+		(shape input)
+		(at 50.8 140.97 180)
+		(fields_autoplaced yes)
+		(effects
+			(font
+				(size 1.27 1.27)
+			)
+			(justify right)
+		)
+		(property "Intersheetrefs" "${INTERSHEET_REFS}"
+			(at 38.6829 140.97 0)
+			(effects
+				(font
+					(size 1.27 1.27)
+				)
+				(justify right)
+				(hide yes)
+			)
+		)
+	)
 	(global_label "RX"
 		(shape input)
@@
 		)
 	)
-	(global_label "A1"
-		(shape input)
-		(at 26.67 64.77 0)
-		(fields_autoplaced yes)
-		(effects
-			(font
-				(size 1.27 1.27)
-			)
-			(justify left)
-		)
-		(property "Intersheetrefs" "${INTERSHEET_REFS}"
-			(at 31.9533 64.77 0)
-			(effects
-				(font
-					(size 1.27 1.27)
-				)
-				(justify left)
-				(hide yes)
-			)
-		)
-	)
-	(global_label "A1"
+	(global_label "DIO0"
 		(shape input)
 		(at 50.8 143.51 180)
@@
 		)
 		(property "Intersheetrefs" "${INTERSHEET_REFS}"
-			(at 45.5167 143.51 0)
+			(at 43.4 143.51 0)
 			(effects
 				(font
@@
 		(property "Intersheetrefs" "${INTERSHEET_REFS}"
 			(at 45.3353 186.69 0)
-			(effects
-				(font
-					(size 1.27 1.27)
-				)
-				(justify right)
-				(hide yes)
-			)
-		)
-	)
-	(global_label "A0"
-		(shape input)
-		(at 26.67 67.31 0)
-		(fields_autoplaced yes)
-		(effects
-			(font
-				(size 1.27 1.27)
-			)
-			(justify left)
-		)
-		(property "Intersheetrefs" "${INTERSHEET_REFS}"
-			(at 31.9533 67.31 0)
-			(effects
-				(font
-					(size 1.27 1.27)
-				)
-				(justify left)
-				(hide yes)
-			)
-		)
-	)
-	(global_label "A0"
-		(shape input)
-		(at 50.8 140.97 180)
-		(fields_autoplaced yes)
-		(effects
-			(font
-				(size 1.27 1.27)
-			)
-			(justify right)
-		)
-		(property "Intersheetrefs" "${INTERSHEET_REFS}"
-			(at 45.5167 140.97 0)
 			(effects
 				(font
@@
 	(symbol
 		(lib_id "power:GND")
-		(at 41.91 138.43 0)
+		(at 35.56 138.43 0)
 		(unit 1)
 		(exclude_from_sim no)
@@
 		(fields_autoplaced yes)
 		(property "Reference" "#PWR014"
-			(at 41.91 144.78 0)
+			(at 35.56 144.78 0)
 			(effects
 				(font
@@
 		)
 		(property "Value" "GND"
-			(at 41.91 143.51 0)
+			(at 35.56 143.51 0)
 			(effects
 				(font
@@
 		)
 		(property "Footprint" ""
-			(at 41.91 138.43 0)
+			(at 35.56 138.43 0)
 			(effects
 				(font
@@
 		)
 		(property "Datasheet" ""
-			(at 41.91 138.43 0)
+			(at 35.56 138.43 0)
 			(effects
 				(font
@@
 		)
 		(property "Description" "Power symbol creates a global label with name \"GND\" , ground"
-			(at 41.91 138.43 0)
-			(effects
-				(font
+			(at 35.56 138.43 0)
+			(effects
+				(font

Commit message: Edit README
Parts:
- U1: value ESP32-C3-MINI-1-N4 -> ESP32-C3-MINI-1-H4; LCSC (none) -> C2934569
Changed lines of the file:
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@@
 			)
 		)
-		(property "Value" "ESP32-C3-MINI-1-N4"
+		(property "Value" "ESP32-C3-MINI-1-H4"
 			(at 71.12 106.68 0)
 			(effects
@@
 			(at 50.8 113.03 0)
 			(effects
+				(font
+					(size 1.27 1.27)
+				)
+				(hide yes)
+			)
+		)
+		(property "LCSC" "C2934569 "
+			(at 50.8 113.03 0)
+			(effects
